Commit message: Update offsets.
Signed-off-by: Benjamin Perseghetti <bperseghetti@rudislabs.com>

File: melm_description/urdf/melm.urdf (robot description, URDF)
Before this commit: robot melm, 4 links, 3 joints
Links:
- link base_link: geometry visual mesh filename=package://melm_description/meshes/HubMotor.dae scale=1 1 1; visual mesh filename=package://melm_description/meshes/HubMotor.dae scale=1 1 1
Joints:
- joint base_joint: origin xyz=0.0 0.0 -.15 rpy=0 0 0 -> xyz=0.0 0.0 -.17 rpy=0 0 0
- joint rplidar_joint: origin xyz=0 0 .22 rpy=0 0 0 -> xyz=0 0 .12 rpy=0 0 0

Commit message: Update launch configs.
Signed-off-by: Benjamin Perseghetti <bperseghetti@rudislabs.com>

File: melm_description/urdf/melm.urdf (robot description, URDF)
Before this commit: robot melm, 4 links, 3 joints
Links:
- removed link /link/rplidar_link/sensor/rplidar/scan
- removed link rplidar_link
- added link /link/lidar_link/sensor/lidar/scan
- added link lidar_link; visual mesh filename=package://melm_description/meshes/STL27L.dae scale=1 1 1
Joints:
- removed joint rplidar_joint
- removed joint rplidar_joint2
- added joint lidar_joint: type fixed, parent base_link, child lidar_link, origin xyz=0 0 .1 rpy=0 0 0
- added joint lidar_joint2: type fixed, parent lidar_link, child /link/lidar_link/sensor/lidar/scan, origin xyz=0.0 0.0 0.0 rpy=0 0 0

Commit message: Updated MELM
Signed-off-by: Benjamin Perseghetti <bperseghetti@rudislabs.com>

File: melm_description/urdf/melm.urdf (robot description, URDF)
Before this commit: robot melm, 4 links, 3 joints
Links:
- removed link /link/lidar_link/sensor/lidar/scan
- link base_link: geometry visual mesh filename=package://melm_description/meshes/HubMotor.dae scale=1 1 1; visual mesh filename=package://melm_description/meshes/HubMotor.dae scale=1 1 1
- link lidar_link: geometry visual box size=0.039 0.039 0.022; visual cylinder length=0.014 radius=0.018
Joints:
- removed joint lidar_joint2
- joint base_joint: origin xyz=0.0 0.0 -.17 rpy=0 0 0 -> xyz=0.0 0.0 0.0 rpy=0 0 0
- joint lidar_joint: origin xyz=0 0 .1 rpy=0 0 0 -> xyz=0 0 0.265 rpy=0 0 0
